File: newloader.kicad_sch (KiCad schematic)
At the start: 44 parts, among them J1 CES, J2 BUTTONS, U1 LTV-847S, U2 LTV-847S, U3 LTV-847S, U4 LTV-847S, U5 LTV-847S

Commit message: V3 for easier parts purchase of 16 pin header
Parts:
- J1: footprint Connector_PinHeader_2.54mm:PinHeader_1x16_P2.54mm_Vertical_SMD_Pin1Left -> Connector_PinHeader_2.54mm:PinHeader_1x16_P2.54mm_Vertical_SMD_Pin1Right
Changed lines of the file:
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@@
       (effects (font (size 1.27 1.27)))
     )
-    (property "Footprint" "Connector_PinHeader_2.54mm:PinHeader_1x16_P2.54mm_Vertical_SMD_Pin1Left" (at 199.39 43.18 0)
+    (property "Footprint" "Connector_PinHeader_2.54mm:PinHeader_1x16_P2.54mm_Vertical_SMD_Pin1Right" (at 199.39 43.18 0)
       (effects (font (size 1.27 1.27)) hide)
     )

Commit message: V4 with alternate wiring to 1130
Prior wiring method allowed bounce to show up as multiple button presses. New method solves that issue.
Parts:
- removed R34: 470, Resistor_SMD:R_0805_2012Metric, symbol Device:R_US
- removed unit 2 of U5
Connections:
- net +12V: no longer U5.12
- net at J2.3 (Pin_3): now also U5.12
Changed lines of the file:
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@@
   (junction (at 132.08 95.25) (diameter 0) (color 0 0 0 0)
   )
-  (junction (at 55.88 24.13) (diameter 0) (color 0 0 0 0)
-  )
   (junction (at 86.36 156.21) (diameter 0) (color 0 0 0 0)
   )
@@
   (junction (at 86.36 100.33) (diameter 0) (color 0 0 0 0)
   )
-  (junction (at 52.07 20.32) (diameter 0) (color 0 0 0 0)
-  )
   (junction (at 207.01 115.57) (diameter 0) (color 0 0 0 0)
   )
@@
   (junction (at 132.08 147.32) (diameter 0) (color 0 0 0 0)
   )
-  (junction (at 77.47 40.64) (diameter 0) (color 0 0 0 0)
-  )
   (junction (at 100.33 39.37) (diameter 0) (color 0 0 0 0)
   )
@@
     (stroke (width 0) (type default))
   )
-  (wire (pts (xy 53.34 29.21) (xy 44.45 29.21))
+  (wire (pts (xy 44.45 29.21) (xy 49.53 29.21))
     (stroke (width 0) (type default))
   )
@@
     (stroke (width 0) (type default))
   )
-  (wire (pts (xy 58.42 35.56) (xy 55.88 35.56))
-    (stroke (width 0) (type default))
-  )
   (wire (pts (xy 198.12 138.43) (xy 190.5 138.43))
     (stroke (width 0) (type default))
@@
     (stroke (width 0) (type default))
   )
+  (wire (pts (xy 49.53 29.21) (xy 49.53 20.32))
+    (stroke (width 0) (type default))
+  )
   (wire (pts (xy 115.57 39.37) (xy 118.11 39.37))
     (stroke (width 0) (type default))
@@
     (stroke (width 0) (type default))
   )
-  (wire (pts (xy 52.07 20.32) (xy 52.07 24.13))
-    (stroke (width 0) (type default))
-  )
-  (wire (pts (xy 52.07 20.32) (xy 33.02 20.32))
-    (stroke (width 0) (type default))
-  )
   (wire (pts (xy 189.23 74.93) (xy 189.23 60.96))
     (stroke (width 0) (type default))
@@
     (stroke (width 0) (type default))
   )
-  (wire (pts (xy 55.88 35.56) (xy 55.88 24.13))
-    (stroke (width 0) (type default))
-  )
   (wire (pts (xy 80.01 139.7) (xy 88.9 139.7))
     (stroke (width 0) (type default))
@@
     (stroke (width 0) (type default))
   )
+  (wire (pts (xy 49.53 20.32) (xy 33.02 20.32))
+    (stroke (width 0) (type default))
+  )
   (wire (pts (xy 91.44 123.19) (xy 91.44 144.78))
     (stroke (width 0) (type default))
@@
     (stroke (width 0) (type default))
   )
-  (wire (pts (xy 53.34 40.64) (xy 53.34 29.21))
-    (stroke (width 0) (type default))
-  )
   (wire (pts (xy 250.19 124.46) (xy 254 124.46))
     (stroke (width 0) (type default))
@@
     (stroke (width 0) (type default))
   )
-  (wire (pts (xy 52.07 19.05) (xy 52.07 20.32))
+  (wire (pts (xy 52.07 19.05) (xy 52.07 24.13))
     (stroke (width 0) (type default))
   )
@@
     (stroke (width 0) (type default))
   )
-  (wire (pts (xy 77.47 40.64) (xy 73.66 40.64))
-    (stroke (width 0) (type default))
-  )
   (wire (pts (xy 92.71 53.34) (xy 88.9 53.34))
     (stroke (width 0) (type default))
@@
   )
   (wire (pts (xy 132.08 53.34) (xy 132.08 67.31))
-    (stroke (width 0) (type default))
-  )
-  (wire (pts (xy 58.42 40.64) (xy 53.34 40.64))
     (stroke (width 0) (type default))
   )
@@
         (path "/738fc3cd-6e95-44b2-a0b7-e799f3451466"
           (reference "R4") (unit 1)
-        )
-      )
-    )
-  )
-  (symbol (lib_id "Device:R_US") (at 77.47 35.56 270) (unit 1)
-    (in_bom yes) (on_board yes) (dnp no) (fields_autoplaced)
-    (property "Reference" "R34" (at 77.47 29.21 90)
-      (effects (font (size 1.27 1.27)))
-    )
-    (property "Value" "470" (at 77.47 31.75 90)
-      (effects (font (size 1.27 1.27)))
-    )
-    (property "Footprint" "Resistor_SMD:R_0805_2012Metric" (at 77.216 36.576 90)
-      (effects (font (size 1.27 1.27)) hide)
-    )
-    (property "Datasheet" "~" (at 77.47 35.56 0)
-      (effects (font (size 1.27 1.27)) hide)
-    )
-    (pin "1")
-    (pin "2")
-    (instances
-      (project "newloader"
-        (path "/738fc3cd-6e95-44b2-a0b7-e799f3451466"
-          (reference "R34") (unit 1)
         )
       )
@@
         )
       )
-    )
-  )
-  (symbol (lib_id "Isolator:LTV-847S") (at 66.04 38.1 0) (mirror y) (unit 2)
-    (in_bom yes) (on_board yes) (dnp no)
-    (property "Reference" "U5" (at 66.04 29.21 0)
-      (effects (font (size 1.27 1.27)))
-    )
-    (property "Value" "LTV-847S" (at 66.04 31.75 0)
-      (effects (font (size 1.27 1.27)))
-    )
-    (property "Footprint" "Package_DIP:SMDIP-16_W9.53mm" (at 66.04 45.72 0)
-      (effects (font (size 1.27 1.27)) hide)
-    )
-    (property "Datasheet" "http://www.us.liteon.com/downloads/LTV-817-827-847.PDF" (at 81.28 26.67 0)
-      (effects (font (size 1.27 1.27)) hide)
-    )
-    (pin "1")
-    (pin "15")
-    (pin "16")
-    (pin "2")
-    (pin "13")
-    (pin "14")
-    (pin "3")
-    (pin "4")
-    (pin "11")
-    (pin "12")
-    (pin "5")
-    (pin "6")
-    (pin "10")
-    (pin "7")
-    (pin "8")
-    (pin "9")
-    (instances
-      (project "newloader"
-        (path "/738fc3cd-6e95-44b2-a0b7-e799f3451466"
-          (reference "U5") (unit 2)
-        )
-      )
